File: pcb/cadpadPCB.kicad_pcb (KiCad board)
At the start: 2 copper layers, 57.2 x 39.9 mm, 6 parts, among them SW1 SW_Push, SW2 SW_Push, SW3 SW_Push, SW4 SW_Push, SW5 SW_Push, U1 XIAO-RP2040-DIP

Commit message: add files!!!!
Routing:
- net Net-(U1-GPIO26/ADC0/A0): track 0.00 -> 51.9 mm
- net Net-(U1-GPIO27/ADC1/A1): track 0.00 -> 39.2 mm
- net Net-(U1-GPIO29/ADC3/A3): track 0.00 -> 26.6 mm
- net Net-(U1-GPIO28/ADC2/A2): track 0.00 -> 21.6 mm
- net Net-(U1-GPIO6/SDA): track 0.00 -> 11.7 mm
Other:
- outline, holes or cut-outs redrawn
- board text added: "Cadpad GingerGigiCat"
- board text added: "XIAO HERE!"
